File: AH3.kicad_pcb (KiCad board)
At the start: 2 copper layers, 29 x 33 mm, 27 parts, among them J1 PROG, J3 I2C, U1 BMP388, U2 BMP388, U3 CH32V305GBU6, Y1 8MHz

Commit message: readme update
Other:
- board text added: "⌀ 2.5"
- board text added: "⌀ 27.0"
- board text added: "⌀ 33.0"
